File: arca-2.0/arca-2.0.brd (EAGLE design)
At the start: 336.6 x 127 mm, 202 parts, among them IC1 MCP6N11R, IC2 MCP6N11R, IC3 MCP6N11R, IC4 MCP6N11R, IC5 LM324D, IC6 LM324D, SW1 1101M2S3CQE2, SW2 1101M2S3CQE2, T1 FQP30N06L, T2 FQP30N06L, T3 FQP30N06L, T4 FQP30N06L, T5 FQP30N06L, T6 FQP30N06L, X1 2540-5

Commit message: heartbeat light
Parts:
- added HBT: (no value), led:CHIPLED_1206
- added R77: 68, rcl:R1206
Connections:
- new net HBT: HBT.A, X1.29
- new net N$75: HBT.C, R77.2
- net GND: now also R77.1
Routing:
- net +5V: track 744.8 -> 0.00 mm, vias 4 -> 0
- net DRV_CTL_1: track 314.2 -> 0.00 mm
- net +10V: track 291.1 -> 0.00 mm, vias 2 -> 0
- net +12V: track 281.5 -> 0.00 mm, vias 2 -> 0
- net DRV_CTL_2: track 280.7 -> 0.00 mm, vias 1 -> 0
- net DRV_CTL_3: track 274.0 -> 0.00 mm, vias 3 -> 0
- net DRV_CTL_6: track 259.2 -> 0.00 mm
- net DRV_CTL_4: track 259.1 -> 0.00 mm, vias 1 -> 0
- net DRV_CTL_5: track 227.4 -> 0.00 mm, vias 1 -> 0
- net SPI_MISO: track 194.4 -> 0.00 mm, vias 4 -> 0
- net SPI_MOSI: track 192.5 -> 0.00 mm, vias 3 -> 0
- net SPI_CLK: track 190.8 -> 0.00 mm, vias 5 -> 0
- net ADC3_CS: track 127.2 -> 0.00 mm, vias 1 -> 0
- net PT1-: track 112.7 -> 0.00 mm, vias 1 -> 0
- net LC4_PREC: track 105.5 -> 0.00 mm, vias 1 -> 0
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
Commit message: found issues with connector orientation
Parts:
- CON_TC1, CON_TC2, CON_TC3, CON_TC4: value LPTA-4POS -> LPTA-3POS; device con-phoenix-5mm:8.2X4 -> con-phoenix-5mm:8.2X3
- moved D4 81.3 mm to (223.5, 43.2), turned to 0 degrees
- moved R22 78.8 mm to (213.4, 12.7), turned to 0 degrees
- moved JP7 78.1 mm to (195.6, 47.0), turned to 90 degrees
- moved R45 76.2 mm to (213.4, 10.2), turned to 180 degrees
- moved FS6 70.0 mm to (219.7, 17.8)
- moved T6 70.0 mm to (223.5, 14.0)
- moved R7 68.7 mm to (262.9, 64.8), turned to 90 degrees
- moved R23 67.9 mm to (233.7, 19.1)
- moved FS_STAT_6 67.9 mm to (240.0, 19.1)
- moved R3 65.6 mm to (265.4, 64.8), turned to 270 degrees
- moved DRV_STAT_6 62.4 mm to (246.4, 17.8)
- moved R24 62.4 mm to (246.4, 11.4)
- moved R10 61.4 mm to (250.2, 64.8), turned to 90 degrees
- moved D10 61.4 mm to (241.3, 11.4)
- moved T1 60.8 mm to (261.6, 73.7)
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Connections:
- net GND: now also CON_TC1.5, CON_TC1.6, CON_TC2.5, CON_TC2.6, CON_TC3.5, CON_TC3.6, CON_TC4.5, CON_TC4.6; no longer CON_TC1.7, CON_TC1.8, CON_TC2.7, CON_TC2.8, CON_TC3.7, CON_TC3.8, CON_TC4.7, CON_TC4.8
Routing:
- net +5V: track 0.00 -> 661.6 mm, vias 0 -> 6
- net +12V: track 0.00 -> 290.0 mm
- net DRV_CTL_2: track 0.00 -> 268.1 mm
- net DRV_CTL_1: track 0.00 -> 260.9 mm
- net +10V: track 0.00 -> 239.9 mm, vias 0 -> 2
- net DRV_CTL_3: track 0.00 -> 234.2 mm, vias 0 -> 1
- net DRV_CTL_4: track 0.00 -> 211.7 mm
- net DRV_CTL_6: track 0.00 -> 189.2 mm, vias 0 -> 1
- net SPI_CLK: track 0.00 -> 188.2 mm, vias 0 -> 4
- net SPI_MISO: track 0.00 -> 186.0 mm, vias 0 -> 3
- net SPI_MOSI: track 0.00 -> 180.5 mm, vias 0 -> 3
- net DRV_CTL_5: track 0.00 -> 165.5 mm, vias 0 -> 2
- net ADC3_CS: track 0.00 -> 118.7 mm, vias 0 -> 1
- net LC4_PREC: track 0.00 -> 110.5 mm, vias 0 -> 1
- net PT1-: track 0.00 -> 99.7 mm, vias 0 -> 2
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Other:
- board size 336.6 x 127 mm -> 276.2 x 127 mm
- board text added: "+5V IN GND"
- board text removed: "+5V VOUT GND"

Commit message: solid model referencing has revealed incorrectly sized connectors
Parts:
- moved PWR_12V 40.4 mm to (215.9, 35.6), turned to 180 degrees
- moved R6 36.1 mm to (215.9, 29.2)
- moved FS7 15.5 mm to (136.1, 91.4)
- moved FS8 15.5 mm to (114.6, 91.4)
- moved FS9 15.5 mm to (93.0, 91.4)
- moved FS10 15.2 mm to (71.1, 91.4)
- moved R8 10.5 mm to (268.0, 86.4)
- moved FS_STAT_1 10.5 mm to (268.0, 92.7)
- moved R11 10.5 mm to (255.3, 86.4)
- moved R14 10.5 mm to (242.6, 86.4)
- moved R17 10.5 mm to (229.9, 86.4)
- moved R20 10.5 mm to (215.9, 86.4)
- moved FS18 10.5 mm to (152.7, 91.4)
- moved FS_STAT_2 10.5 mm to (255.3, 92.7)
- moved FS_STAT_3 10.5 mm to (242.6, 92.7)
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Routing:
- net +5V: track 661.6 -> 0.00 mm, vias 6 -> 0
- net +12V: track 290.0 -> 0.00 mm
- net DRV_CTL_2: track 268.1 -> 0.00 mm
- net DRV_CTL_1: track 260.9 -> 0.00 mm
- net +10V: track 239.9 -> 0.00 mm, vias 2 -> 0
- net DRV_CTL_3: track 234.2 -> 0.00 mm, vias 1 -> 0
- net DRV_CTL_4: track 211.7 -> 0.00 mm
- net DRV_CTL_6: track 189.2 -> 0.00 mm, vias 1 -> 0
- net SPI_CLK: track 188.2 -> 0.00 mm, vias 4 -> 0
- net SPI_MISO: track 186.0 -> 0.00 mm, vias 3 -> 0
- net SPI_MOSI: track 180.5 -> 0.00 mm, vias 3 -> 0
- net DRV_CTL_5: track 165.5 -> 0.00 mm, vias 2 -> 0
- net ADC3_CS: track 118.7 -> 0.00 mm, vias 1 -> 0
- net LC4_PREC: track 110.5 -> 0.00 mm, vias 1 -> 0
- net PT1-: track 99.7 -> 0.00 mm, vias 2 -> 0
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Other:
- board text removed: "+"
- board text removed: "+ -"
- board text removed: "+12V"
- board text removed: "+5V + - GND"
- board text removed: "+5V IN GND"
- board text removed: "-"
- board text removed: "GND"

Commit message: bigger 5mm connectors
Parts:
- moved R5 52.1 mm to (196.8, 33.0), turned to 270 degrees
- moved PWR_10V 47.9 mm to (196.8, 26.7), turned to 0 degrees
- moved R75 47.2 mm to (67.3, 27.9), turned to 0 degrees
- moved C28 44.2 mm to (67.3, 36.8), turned to 0 degrees
- moved JP6 44.0 mm to (154.9, 26.7), turned to 90 degrees
- moved D3 42.2 mm to (195.6, 12.7), turned to 270 degrees
- moved JP2 42.1 mm to (101.6, 33.0), turned to 90 degrees
- moved C5 40.7 mm to (190.5, 27.9), turned to 180 degrees
- moved R34 40.4 mm to (148.6, 35.6), turned to 180 degrees
- moved D4 37.0 mm to (260.4, 39.4)
- moved JP7 34.9 mm to (228.6, 35.6)
- moved R30 34.3 mm to (148.6, 17.8), turned to 180 degrees
- moved R36 34.3 mm to (141.0, 38.1), turned to 270 degrees
- moved C6 34.2 mm to (189.2, 7.62), turned to 180 degrees
- moved ADC2 33.5 mm to (58.4, 31.8), turned to 270 degrees
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Other:
- board size 276.2 x 127 mm -> 292.1 x 114.3 mm

Commit message: routing on shrunken board
Routing:
- net +5V: track 0.00 -> 620.1 mm, vias 0 -> 4
- net +10V: track 0.00 -> 287.1 mm, vias 0 -> 2
- net +12V: track 0.00 -> 282.1 mm
- net DRV_CTL_1: track 0.00 -> 281.1 mm, vias 0 -> 1
- net DRV_CTL_2: track 0.00 -> 261.5 mm
- net DRV_CTL_3: track 0.00 -> 244.1 mm, vias 0 -> 1
- net DRV_CTL_4: track 0.00 -> 212.1 mm
- net DRV_CTL_5: track 0.00 -> 182.0 mm
- net DRV_CTL_6: track 0.00 -> 164.5 mm, vias 0 -> 1
- net SPI_MISO: track 0.00 -> 149.6 mm, vias 0 -> 4
- net SPI_MOSI: track 0.00 -> 141.4 mm, vias 0 -> 3
- net SPI_CLK: track 0.00 -> 139.9 mm, vias 0 -> 5
- net LC4_PREC: track 0.00 -> 113.5 mm, vias 0 -> 2
- net ADC3_CS: track 0.00 -> 111.5 mm, vias 0 -> 1
- net LC1_PREC: track 0.00 -> 105.6 mm
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
Commit message: final revisions on board before design review
Parts:
- moved R71 1.27 mm to (19.1, 52.1)
- moved D9 1.27 mm to (226.1, 80.0)
- moved FS10 1.27 mm to (76.2, 77.5)
- moved FS11 1.27 mm to (53.3, 77.5)
- moved FS12 1.27 mm to (40.6, 77.5)
- moved FS13 1.27 mm to (27.9, 77.5)
- moved FS14 1.27 mm to (15.2, 77.5)
- moved FS17 1.27 mm to (180.6, 77.5)
- moved FS18 1.27 mm to (162.8, 77.5)
- moved FS7 1.27 mm to (145.0, 77.5)
- moved FS8 1.27 mm to (122.2, 77.5)
- moved FS9 1.27 mm to (99.3, 77.5)
Routing:
- net +5V: track 620.1 -> 584.9 mm
- net +10V: track 287.1 -> 273.6 mm
- net DRV_CTL_4: track 212.1 -> 200.6 mm, vias 0 -> 1
- net TC2: track 58.9 -> 56.5 mm
- net DRV_CTL_1: track 281.1 -> 278.9 mm
- net DRV_CTL_5: track 182.0 -> 180.5 mm
- net DRV_CTL_6: track 164.5 -> 163.1 mm
- net TC1: track 70.4 -> 69.1 mm
- net N$70: track 31.6 -> 32.9 mm
- net N$65: track 31.6 -> 32.9 mm
- net N$64: track 31.7 -> 32.9 mm
- net DRV_NEG_5: track 55.0 -> 56.3 mm
- net N$69: track 31.6 -> 32.9 mm
- net N$66: track 31.6 -> 32.9 mm
- net N$74: track 30.3 -> 31.6 mm
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Other:
- board text added: "4- 4+ 3- 3+ 2- 2+ 1- 1+"
- board text added: "ARCA 2.0"
- board text added: "DRV6 DRV5 DRV4 DRV3 DRV2 DRV1"
- board text added: "Designed with <3 by"
- board text added: "LC4 LC3 LC2 LC1"
- board text added: "PT1 PT2 PT3 PT4"
- board text added: "PT4- PT3- PT2- PT1-"
- board text added: "RICE ECLIPSE"
- board text added: "TC4 TC3 TC2 TC1"

Commit message: values tweaks as we make a BOM
Parts:
- DRV_STAT_1, DRV_STAT_2, DRV_STAT_3, DRV_STAT_4, DRV_STAT_5, DRV_STAT_6: value (none) -> YLW
- FS_STAT_1, FS_STAT_2, FS_STAT_3, FS_STAT_4, FS_STAT_5, FS_STAT_6, HBT: value (none) -> BLU
Changed lines of the file:
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@@
 <attribute name="VALUE" x="285.75" y="72.39" size="1.27" layer="27" rot="R90"/>
 </element>
-<element name="FS_STAT_1" library="led" library_urn="urn:adsk.eagle:library:259" package="CHIPLED_1206" package3d_urn="urn:adsk.eagle:package:15823/2" value="" x="283.21" y="80.01" smashed="yes" rot="R180">
+<element name="FS_STAT_1" library="led" library_urn="urn:adsk.eagle:library:259" package="CHIPLED_1206" package3d_urn="urn:adsk.eagle:package:15823/2" value="BLU" x="283.21" y="80.01" smashed="yes" rot="R180">
 <attribute name="NAME" x="284.48" y="82.55" size="1.27" layer="25" rot="R270"/>
 <attribute name="POPULARITY" value="28" x="283.21" y="80.01" size="1.778" layer="27" rot="R180" display="off"/>
@@
 <attribute name="VALUE" x="275.59" y="83.82" size="1.27" layer="27"/>
 </element>
-<element name="DRV_STAT_1" library="led" library_urn="urn:adsk.eagle:library:259" package="CHIPLED_1206" package3d_urn="urn:adsk.eagle:package:15823/2" value="" x="283.21" y="86.36" smashed="yes" rot="R90">
+<element name="DRV_STAT_1" library="led" library_urn="urn:adsk.eagle:library:259" package="CHIPLED_1206" package3d_urn="urn:adsk.eagle:package:15823/2" value="YLW" x="283.21" y="86.36" smashed="yes" rot="R90">
 <attribute name="NAME" x="285.75" y="85.09" size="1.27" layer="25" rot="R180"/>
 <attribute name="POPULARITY" value="28" x="283.21" y="86.36" size="1.778" layer="27" rot="R90" display="off"/>
@@
 <attribute name="VALUE" x="273.05" y="72.39" size="1.27" layer="27" rot="R90"/>
 </element>
-<element name="FS_STAT_2" library="led" library_urn="urn:adsk.eagle:library:259" package="CHIPLED_1206" package3d_urn="urn:adsk.eagle:package:15823/2" value="" x="270.51" y="80.01" smashed="yes" rot="R180">
+<element name="FS_STAT_2" library="led" library_urn="urn:adsk.eagle:library:259" package="CHIPLED_1206" package3d_urn="urn:adsk.eagle:package:15823/2" value="BLU" x="270.51" y="80.01" smashed="yes" rot="R180">
 <attribute name="NAME" x="271.78" y="82.55" size="1.27" layer="25" rot="R270"/>
 <attribute name="POPULARITY" value="28" x="278.13" y="72.39" size="1.778" layer="27" rot="R180" display="off"/>
@@
 <attribute name="VALUE" x="262.89" y="83.82" size="1.27" layer="27"/>
 </element>
-<element name="DRV_STAT_2" library="led" library_urn="urn:adsk.eagle:library:259" package="CHIPLED_1206" package3d_urn="urn:adsk.eagle:package:15823/2" value="" x="270.51" y="86.36" smashed="yes" rot="R90">
+<element name="DRV_STAT_2" library="led" library_urn="urn:adsk.eagle:library:259" package="CHIPLED_1206" package3d_urn="urn:adsk.eagle:package:15823/2" value="YLW" x="270.51" y="86.36" smashed="yes" rot="R90">
 <attribute name="NAME" x="273.05" y="85.09" size="1.27" layer="25" rot="R180"/>
 <attribute name="POPULARITY" value="28" x="293.37" y="72.39" size="1.778" layer="27" rot="R90" display="off"/>
@@
 <attribute name="VALUE" x="260.35" y="72.39" size="1.27" layer="27" rot="R90"/>
 </element>
-<element name="FS_STAT_3" library="led" library_urn="urn:adsk.eagle:library:259" package="CHIPLED_1206" package3d_urn="urn:adsk.eagle:package:15823/2" value="" x="257.81" y="80.01" smashed="yes" rot="R180">
+<element name="FS_STAT_3" library="led" library_urn="urn:adsk.eagle:library:259" package="CHIPLED_1206" package3d_urn="urn:adsk.eagle:package:15823/2" value="BLU" x="257.81" y="80.01" smashed="yes" rot="R180">
 <attribute name="NAME" x="259.08" y="82.55" size="1.27" layer="25" rot="R270"/>
 <attribute name="POPULARITY" value="28" x="265.43" y="72.39" size="1.778" layer="27" rot="R180" display="off"/>
@@
 <attribute name="VALUE" x="248.92" y="83.82" size="1.27" layer="27"/>
 </element>
-<element name="DRV_STAT_3" library="led" library_urn="urn:adsk.eagle:library:259" package="CHIPLED_1206" package3d_urn="urn:adsk.eagle:package:15823/2" value="" x="256.54" y="86.36" smashed="yes" rot="R90">
+<element name="DRV_STAT_3" library="led" library_urn="urn:adsk.eagle:library:259" package="CHIPLED_1206" package3d_urn="urn:adsk.eagle:package:15823/2" value="YLW" x="256.54" y="86.36" smashed="yes" rot="R90">
 <attribute name="NAME" x="260.35" y="85.09" size="1.27" layer="25" rot="R180"/>
 <attribute name="POPULARITY" value="28" x="279.4" y="72.39" size="1.778" layer="27" rot="R90" display="off"/>
@@
 <attribute name="VALUE" x="247.65" y="72.39" size="1.27" layer="27" rot="R90"/>
 </element>
-<element name="FS_STAT_4" library="led" library_urn="urn:adsk.eagle:library:259" package="CHIPLED_1206" package3d_urn="urn:adsk.eagle:package:15823/2" value="" x="245.11" y="80.01" smashed="yes" rot="R180">
+<element name="FS_STAT_4" library="led" library_urn="urn:adsk.eagle:library:259" package="CHIPLED_1206" package3d_urn="urn:adsk.eagle:package:15823/2" value="BLU" x="245.11" y="80.01" smashed="yes" rot="R180">
 <attribute name="NAME" x="246.38" y="82.55" size="1.27" layer="25" rot="R270"/>
 <attribute name="POPULARITY" value="28" x="298.45" y="73.66" size="1.778" layer="27" rot="R180" display="off"/>
@@
 <attribute name="VALUE" x="236.22" y="83.82" size="1.27" layer="27"/>
 </element>
-<element name="DRV_STAT_4" library="led" library_urn="urn:adsk.eagle:library:259" package="CHIPLED_1206" package3d_urn="urn:adsk.eagle:package:15823/2" value="" x="243.84" y="86.36" smashed="yes" rot="R90">
+<element name="DRV_STAT_4" library="led" library_urn="urn:adsk.eagle:library:259" package="CHIPLED_1206" package3d_urn="urn:adsk.eagle:package:15823/2" value="YLW" x="243.84" y="86.36" smashed="yes" rot="R90">
 <attribute name="NAME" x="247.65" y="85.09" size="1.27" layer="25" rot="R180"/>
 <attribute name="POPULARITY" value="28" x="267.97" y="72.39" size="1.778" layer="27" rot="R90" display="off"/>
@@
 <attribute name="VALUE" x="233.68" y="72.39" size="1.27" layer="27" rot="R90"/>
 </element>
-<element name="FS_STAT_5" library="led" library_urn="urn:adsk.eagle:library:259" package="CHIPLED_1206" package3d_urn="urn:adsk.eagle:package:15823/2" value="" x="231.14" y="80.01" smashed="yes" rot="R180">
+<element name="FS_STAT_5" library="led" library_urn="urn:adsk.eagle:library:259" package="CHIPLED_1206" package3d_urn="urn:adsk.eagle:package:15823/2" value="BLU" x="231.14" y="80.01" smashed="yes" rot="R180">
 <attribute name="NAME" x="232.41" y="82.55" size="1.27" layer="25" rot="R270"/>
 <attribute name="POPULARITY" value="28" x="251.46" y="118.11" size="1.778" layer="27" rot="R180" display="off"/>
@@
 <attribute name="VALUE" x="223.52" y="83.82" size="1.27" layer="27"/>
 </element>
-<element name="DRV_STAT_5" library="led" library_urn="urn:adsk.eagle:library:259" package="CHIPLED_1206" package3d_urn="urn:adsk.eagle:package:15823/2" value="" x="231.14" y="86.36" smashed="yes" rot="R90">
+<element name="DRV_STAT_5" library="led" library_urn="urn:adsk.eagle:library:259" package="CHIPLED_1206" package3d_urn="urn:adsk.eagle:package:15823/2" value="YLW" x="231.14" y="86.36" smashed="yes" rot="R90">
 <attribute name="NAME" x="233.68" y="85.09" size="1.27" layer="25" rot="R180"/>
 <attribute name="POPULARITY" value="28" x="312.42" y="54.61" size="1.778" layer="27" rot="R90" display="off"/>
@@
 <attribute name="VALUE" x="228.6" y="11.43" size="1.27" layer="27"/>
 </element>
-<element name="FS_STAT_6" library="led" library_urn="urn:adsk.eagle:library:259" package="CHIPLED_1206" package3d_urn="urn:adsk.eagle:package:15823/2" value="" x="236.22" y="13.97" smashed="yes" rot="R90">
+<element name="FS_STAT_6" library="led" library_urn="urn:adsk.eagle:library:259" package="CHIPLED_1206" package3d_urn="urn:adsk.eagle:package:15823/2" value="BLU" x="236.22" y="13.97" smashed="yes" rot="R90">
 <attribute name="NAME" x="238.76" y="12.7" size="1.27" layer="25" rot="R180"/>
 <attribute name="POPULARITY" value="28" x="331.47" y="-24.13" size="1.778" layer="27" rot="R90" display="off"/>
@@
 <attribute name="VALUE" x="240.03" y="22.86" size="1.27" layer="27" rot="R270"/>
 </element>
-<element name="DRV_STAT_6" library="led" library_urn="urn:adsk.eagle:library:259" package="CHIPLED_1206" package3d_urn="urn:adsk.eagle:package:15823/2" value="" x="242.57" y="15.24" smashed="yes">
+<element name="DRV_STAT_6" library="led" library_urn="urn:adsk.eagle:library:259" package="CHIPLED_1206" package3d_urn="urn:adsk.eagle:package:15823/2" value="YLW" x="242.57" y="15.24" smashed="yes">
 <attribute name="NAME" x="241.3" y="12.7" size="1.27" layer="25" rot="R90"/>
 <attribute name="POPULARITY" value="28" x="193.04" y="-123.19" size="1.778" layer="27" display="off"/>
@@
 <attribute name="VALUE" x="157.814" y="86.47" size="1.27" layer="27" rot="R270"/>
 </element>
-<element name="HBT" library="led" library_urn="urn:adsk.eagle:library:259" package="CHIPLED_1206" package3d_urn="urn:adsk.eagle:package:15823/2" value="" x="76.2" y="29.21" smashed="yes">
+<element name="HBT" library="led" library_urn="urn:adsk.eagle:library:259" package="CHIPLED_1206" package3d_urn="urn:adsk.eagle:package:15823/2" value="BLU" x="76.2" y="29.21" smashed="yes">
 <attribute name="NAME" x="74.93" y="27.94" size="1.27" layer="25" rot="R90"/>
 <attribute name="POPULARITY" value="28" x="68.58" y="41.91" size="1.778" layer="27" display="off"/>

Commit message: slight reshaping of schematic to make more human-readable
Parts:
- C27, C28, C29: value 0.1u -> 100n
Changed lines of the file:
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@@
 <attribute name="VALUE" x="94.615" y="39.497" size="1.27" layer="27" rot="R180"/>
 </element>
-<element name="C27" library="rcl" library_urn="urn:adsk.eagle:library:334" package="C1206" package3d_urn="urn:adsk.eagle:package:23618/2" value="0.1u" x="83.82" y="27.94" smashed="yes" rot="R180">
+<element name="C27" library="rcl" library_urn="urn:adsk.eagle:library:334" package="C1206" package3d_urn="urn:adsk.eagle:package:23618/2" value="100n" x="83.82" y="27.94" smashed="yes" rot="R180">
 <attribute name="NAME" x="85.09" y="26.67" size="1.27" layer="25" rot="R180"/>
 <attribute name="POPULARITY" value="24" x="83.82" y="27.94" size="1.778" layer="27" rot="R180" display="off"/>
@@
 <attribute name="VALUE" x="56.515" y="25.273" size="1.27" layer="27"/>
 </element>
-<element name="C28" library="rcl" library_urn="urn:adsk.eagle:library:334" package="C1206" package3d_urn="urn:adsk.eagle:package:23618/2" value="0.1u" x="67.31" y="36.83" smashed="yes">
+<element name="C28" library="rcl" library_urn="urn:adsk.eagle:library:334" package="C1206" package3d_urn="urn:adsk.eagle:package:23618/2" value="100n" x="67.31" y="36.83" smashed="yes">
 <attribute name="NAME" x="66.04" y="38.1" size="1.27" layer="25"/>
 <attribute name="POPULARITY" value="24" x="67.31" y="34.29" size="1.778" layer="27" display="off"/>
@@
 <attribute name="VALUE" x="164.973" y="56.515" size="1.27" layer="27" rot="R270"/>
 </element>
-<element name="C29" library="rcl" library_urn="urn:adsk.eagle:library:334" package="C1206" package3d_urn="urn:adsk.eagle:package:23618/2" value="0.1u" x="176.53" y="46.99" smashed="yes" rot="R270">
+<element name="C29" library="rcl" library_urn="urn:adsk.eagle:library:334" package="C1206" package3d_urn="urn:adsk.eagle:package:23618/2" value="100n" x="176.53" y="46.99" smashed="yes" rot="R270">
 <attribute name="NAME" x="177.8" y="48.26" size="1.27" layer="25" rot="R270"/>
 <attribute name="POPULARITY" value="24" x="173.99" y="46.99" size="1.778" layer="27" rot="R270" display="off"/>
